Commit message: "模型已改，重新训练"

File: source/robot_lab/data/Robots/helios_leg/urdf/LW-360 Gen2V1.urdf (robot description, URDF)
Before this commit: robot LW-360 Gen2V1, 7 links, 6 joints
Links:
- link base_link: geometry collision box size=0.46 0.24 0.18; collision cylinder length=0.08 radius=0.05
- link left_calf_link: mass 0.29257 -> 0.3123662; geometry collision cylinder length=0.02 radius=0.02; collision cylinder length=0.06 radius=0.03
- link left_foot_link: geometry collision cylinder length=0.04 radius=0.05; visual mesh filename=meshes/left_foot_link.STL
- link left_thigh_link: mass 0.29712 -> 0.610696054077469; geometry collision cylinder length=0.1 radius=0.035; collision cylinder length=0.2 radius=0.025
- link right_calf_link: geometry collision cylinder length=0.02 radius=0.02; collision cylinder length=0.06 radius=0.03
- link right_foot_link: geometry collision cylinder length=0.04 radius=0.05; visual mesh filename=meshes/right_foot_link.STL
- link right_thigh_link: geometry collision cylinder length=0.1 radius=0.035; collision cylinder length=0.2 radius=0.025

Commit message: “改bug”

File: source/robot_lab/data/Robots/helios_leg/urdf/LW-360 Gen2V1.urdf (robot description, URDF)
Before this commit: robot LW-360 Gen2V1, 7 links, 6 joints
Joints:
- joint left_calf_joint: origin xyz=-0.0331636364235269 0.0174999999999982 0.212426865577748 rpy=0 0 0 -> xyz=-0.0331636364236594 0.0184999999999837 0.212426865577682 rpy=0 0 0
- joint left_thigh_joint: origin xyz=-0.0337728171222443 0.165388304832666 -0.0275000000000591 rpy=0 0 0 -> xyz=-0.0337728171221104 0.164614695167351 -0.0274999999999989 rpy=0 0 0
